Commit message: control cinematico listo

File: fanuc_robot/fanuc_lrmate200id_support/urdf/lrmate200id_macro.xacro (robot description, xacro)
@@ -3,6 +3,12 @@
   <xacro:include filename="$(find fanuc_resources)/urdf/common_materials.xacro"/>
   <xacro:macro name="fanuc_lrmate200id" params="prefix">
+    <link name="world" />
     <!-- links: main serial chain -->
     <link name="${prefix}base_link">
+      <inertial>
+        <origin xyz="0 0 0" rpy="0 0 0"/>
+        <mass value="2.0"/>
+        <inertia ixx="0.01" ixy="0.0" ixz="0.0" iyy="0.01" iyz="0.0" izz="0.01"/>
+      </inertial>
       <visual>
         <origin xyz="0 0 0" rpy="0 0 0"/>
@@ -20,4 +26,9 @@
     </link>
     <link name="${prefix}link_1">
+      <inertial>
+        <origin xyz="0 0 0" rpy="0 0 0"/>
+        <mass value="1.5"/>
+        <inertia ixx="0.01" ixy="0.0" ixz="0.0" iyy="0.01" iyz="0.0" izz="0.01"/>
+      </inertial>
       <visual>
         <origin xyz="0 0 0" rpy="0 0 0"/>
@@ -35,4 +46,9 @@
     </link>
     <link name="${prefix}link_2">
+      <inertial>
+        <origin xyz="0 0 0" rpy="0 0 0"/>
+        <mass value="1.2"/>
+        <inertia ixx="0.01" ixy="0.0" ixz="0.0" iyy="0.01" iyz="0.0" izz="0.01"/>
+      </inertial>
       <visual>
         <origin xyz="0 0 0" rpy="0 0 0"/>
@@ -50,4 +66,9 @@
     </link>
     <link name="${prefix}link_3">
+      <inertial>
+        <origin xyz="0 0 0" rpy="0 0 0"/>
+        <mass value="1.0"/>
+        <inertia ixx="0.01" ixy="0.0" ixz="0.0" iyy="0.01" iyz="0.0" izz="0.01"/>
+      </inertial>
       <visual>
         <origin xyz="0 0 0" rpy="0 0 0"/>
@@ -65,4 +86,9 @@
     </link>
     <link name="${prefix}link_4">
+      <inertial>
+        <origin xyz="0 0 0" rpy="0 0 0"/>
+        <mass value="0.8"/>
+        <inertia ixx="0.01" ixy="0.0" ixz="0.0" iyy="0.01" iyz="0.0" izz="0.01"/>
+      </inertial>
       <visual>
         <origin xyz="0 0 0" rpy="0 0 0"/>
@@ -80,4 +106,9 @@
     </link>
     <link name="${prefix}link_5">
+      <inertial>
+        <origin xyz="0 0 0" rpy="0 0 0"/>
+        <mass value="0.6"/>
+        <inertia ixx="0.01" ixy="0.0" ixz="0.0" iyy="0.01" iyz="0.0" izz="0.01"/>
+      </inertial>
       <visual>
         <origin xyz="0 0 0" rpy="0 0 0"/>
@@ -95,4 +126,9 @@
     </link>
     <link name="${prefix}link_6">
+      <inertial>
+        <origin xyz="0 0 0" rpy="0 0 0"/>
+        <mass value="0.5"/>
+        <inertia ixx="0.01" ixy="0.0" ixz="0.0" iyy="0.01" iyz="0.0" izz="0.01"/>
+      </inertial>
       <visual>
         <origin xyz="0 0 0" rpy="0 0 0"/>
@@ -115,5 +151,5 @@
       <child link="${prefix}link_1" />
       <axis xyz="0 0 1" />
-      <limit effort="0" lower="${radians(-170)}" upper="${radians(170)}" velocity="${radians(450)}" />
+      <limit effort="30" lower="${radians(-170)}" upper="${radians(170)}" velocity="${radians(450)}" />
     </joint>
     <joint name="${prefix}joint_2" type="revolute">
@@ -122,5 +158,5 @@
       <child link="${prefix}link_2" />
       <axis xyz="0 1 0" />
-      <limit effort="0" lower="${radians(-100)}" upper="${radians(145)}" velocity="${radians(380)}" />
+      <limit effort="30" lower="${radians(-100)}" upper="${radians(145)}" velocity="${radians(380)}" />
     </joint>
     <joint name="${prefix}joint_3" type="revolute">
@@ -129,5 +165,5 @@
       <child link="${prefix}link_3" />
       <axis xyz="0 -1 0" />
-      <limit effort="0" lower="${radians(-70)}" upper="${radians(205)}" velocity="${radians(520)}" />
+      <limit effort="30" lower="${radians(-70)}" upper="${radians(205)}" velocity="${radians(520)}" />
     </joint>
     <joint name="${prefix}joint_4" type="revolute">
@@ -136,5 +172,5 @@
       <child link="${prefix}link_4"/>
       <axis xyz="-1 0 0"/>
-      <limit effort="0" lower="${radians(-190)}" upper="${radians(190)}" velocity="${radians(550)}" />
+      <limit effort="20" lower="${radians(-190)}" upper="${radians(190)}" velocity="${radians(550)}" />
     </joint>
     <joint name="${prefix}joint_5" type="revolute">
@@ -143,5 +179,5 @@
       <child link="${prefix}link_5"/>
       <axis xyz="0 -1 0"/>
-      <limit effort="0" lower="${radians(-125)}" upper="${radians(125)}" velocity="${radians(545)}" />
+      <limit effort="20" lower="${radians(-125)}" upper="${radians(125)}" velocity="${radians(545)}" />
     </joint>
     <joint name="${prefix}joint_6" type="revolute">
@@ -150,7 +186,7 @@
       <child link="${prefix}link_6"/>
       <axis xyz="-1 0 0"/>
-      <limit effort="0" lower="${radians(-360)}" upper="${radians(360)}" velocity="${radians(1000)}" />
-    </joint>
-    <!-- ROS-Industrial 'base' frame: base_link to Fanuc World Coordinates transform -->
+      <limit effort="10" lower="${radians(-360)}" upper="${radians(360)}" velocity="${radians(1000)}" />
+    </joint>
+    <!-- ROS-Industrial 'base' frame -->
     <link name="${prefix}base" />
     <joint name="${prefix}base_link-base" type="fixed">
@@ -159,5 +195,5 @@
       <child link="${prefix}base"/>
     </joint>
-    <!-- ROS-Industrial 'flange' frame: attachment point for EEF models -->
+    <!-- 'flange' and 'tool0' -->
     <link name="${prefix}flange" />
     <joint name="${prefix}link_6-flange" type="fixed">
@@ -166,5 +202,4 @@
       <child link="${prefix}flange" />
     </joint>
-    <!-- ROS-Industrial 'tool0' frame: all-zeros tool frame -->
     <link name="${prefix}tool0" />
     <joint name="${prefix}flange-tool0" type="fixed">
@@ -173,4 +208,75 @@
       <child link="${prefix}tool0" />
     </joint>
+    <!-- Gazebo ROS Control Plugin -->
+    <gazebo>
+      <plugin name="gazebo_ros_control" filename="libgazebo_ros_control.so">
+        <robotNamespace>/</robotNamespace>
+      </plugin>
+    </gazebo>
+    <!-- Transmissions -->
+    <transmission name="${prefix}trans_joint_1">
+      <type>transmission_interface/SimpleTransmission</type>
+      <joint name="${prefix}joint_1">
+        <hardwareInterface>hardware_interface/PositionJointInterface</hardwareInterface>
+      </joint>
+      <actuator name="${prefix}motor_joint_1">
+        <mechanicalReduction>1</mechanicalReduction>
+      </actuator>
+    </transmission>
+    <!-- Repite para los demás joints -->
+    <transmission name="${prefix}trans_joint_2">
+      <type>transmission_interface/SimpleTransmission</type>
+      <joint name="${prefix}joint_2">
+        <hardwareInterface>hardware_interface/PositionJointInterface</hardwareInterface>
+      </joint>
+      <actuator name="${prefix}motor_joint_2">
+        <mechanicalReduction>1</mechanicalReduction>
+      </actuator>
+    </transmission>
+    <transmission name="${prefix}trans_joint_3">
+      <type>transmission_interface/SimpleTransmission</type>
+      <joint name="${prefix}joint_3">
+        <hardwareInterface>hardware_interface/PositionJointInterface</hardwareInterface>
+      </joint>
+      <actuator name="${prefix}motor_joint_3">
+        <mechanicalReduction>1</mechanicalReduction>
+      </actuator>
+    </transmission>
+    <transmission name="${prefix}trans_joint_4">
+      <type>transmission_interface/SimpleTransmission</type>
+      <joint name="${prefix}joint_4">
+        <hardwareInterface>hardware_interface/PositionJointInterface</hardwareInterface>
+      </joint>
+      <actuator name="${prefix}motor_joint_4">
+        <mechanicalReduction>1</mechanicalReduction>
+      </actuator>
+    </transmission>
+    <transmission name="${prefix}trans_joint_5">
+      <type>transmission_interface/SimpleTransmission</type>
+      <joint name="${prefix}joint_5">
+        <hardwareInterface>hardware_interface/PositionJointInterface</hardwareInterface>
+      </joint>
+      <actuator name="${prefix}motor_joint_5">
+        <mechanicalReduction>1</mechanicalReduction>
+      </actuator>
+    </transmission>
+    <transmission name="${prefix}trans_joint_6">
+      <type>transmission_interface/SimpleTransmission</type>
+      <joint name="${prefix}joint_6">
+        <hardwareInterface>hardware_interface/PositionJointInterface</hardwareInterface>
+      </joint>
+      <actuator name="${prefix}motor_joint_6">
+        <mechanicalReduction>1</mechanicalReduction>
+      </actuator>
+    </transmission>
+    <!-- Anchor to Gazebo world -->
+    <gazebo reference="${prefix}base_link">
+      <pose>0 0 0 0 0 0</pose>
+    </gazebo>
+    <joint name="${prefix}world_joint" type="fixed">
+      <parent link="world"/>
+      <child link="${prefix}base_link"/>
+      <origin xyz="0 0 0" rpy="0 0 0"/>
+    </joint>
   </xacro:macro>
 </robot>

Commit message: gripper agregado

File: fanuc_robot/fanuc_lrmate200id_support/urdf/lrmate200id_macro.xacro (robot description, xacro)
@@ -202,4 +202,96 @@
       <child link="${prefix}flange" />
     </joint>
+    <!-- Gripper base -->
+    <link name="${prefix}gripper_base">
+      <visual>
+        <origin xyz="0.0 0 0" rpy="0 0 0"/>
+        <geometry>
+          <box size="0.02 0.2 0.05"/>
+        </geometry>
+        <material name="gray">
+          <color rgba="0.5 0.5 0.5 1.0"/>
+        </material>
+      </visual>
+      <collision>
+        <origin xyz="0.0 0 0" rpy="0 0 0"/>
+        <geometry>
+          <box size="0.02 0.2 0.05"/>
+        </geometry>
+      </collision>
+    </link>
+    <gazebo reference="${prefix}gripper_base">
+      <material>Gazebo/Grey</material>
+    </gazebo>
+    <joint name="${prefix}link_6-gripper_base" type="fixed">
+      <origin xyz="0 0 0" rpy="0 0 0"/>
+      <parent link="${prefix}link_6"/>
+      <child link="${prefix}gripper_base"/>
+    </joint>
+    <!-- Dedo izquierdo (finger_1) -->
+    <link name="${prefix}finger_1">
+      <inertial>
+        <origin xyz="0.05 0 0" rpy="0 0 0"/>
+        <mass value="0.1"/>
+        <inertia ixx="1e-4" ixy="0" ixz="0" iyy="1e-4" iyz="0" izz="1e-4"/>
+      </inertial>
+      <visual>
+        <origin xyz="0.03 0.037 0.001" rpy="0 0 0"/>
+        <geometry>
+          <box size="0.10 0.02 0.03"/>
+        </geometry>
+        <material name="gray">
+          <color rgba="0.5 0.5 0.5 1.0"/>
+        </material>
+      </visual>
+      <collision>
+        <origin xyz="0.03 0.037 0.001" rpy="0 0 0"/>
+        <geometry>
+          <box size="0.10 0.02 0.03"/>
+        </geometry>
+      </collision>
+    </link>
+    <gazebo reference="${prefix}finger_1">
+      <material>Gazebo/Grey</material>
+    </gazebo>
+    <joint name="${prefix}gripper_base_finger_1" type="prismatic">
+      <origin xyz="0.03 0.037 0.001" rpy="0 0 0"/>
+      <parent link="${prefix}gripper_base"/>
+      <child link="${prefix}finger_1"/>
+      <axis xyz="0 -1 0"/>   <!-- Cambia a -1 -->
+      <limit effort="1.0" lower="0" upper="0.04" velocity="0.1"/>
+    </joint>
+    <!-- Dedo derecho (finger_2) -->
+    <link name="${prefix}finger_2">
+      <inertial>
+        <origin xyz="0.05 0 0" rpy="0 0 0"/>
+        <mass value="0.1"/>
+        <inertia ixx="1e-4" ixy="0" ixz="0" iyy="1e-4" iyz="0" izz="1e-4"/>
+      </inertial>
+      <visual>
+        <origin xyz="0.03 -0.037 0.001" rpy="0 0 0"/>
+        <geometry>
+          <box size="0.10 0.02 0.03"/>
+        </geometry>
+        <material name="gray">
+          <color rgba="0.5 0.5 0.5 1.0"/>
+        </material>
+      </visual>
+      <collision>
+        <origin xyz="0.03 -0.037 0.001" rpy="0 0 0"/>
+        <geometry>
+          <box size="0.10 0.02 0.03"/>
+        </geometry>
+      </collision>
+    </link>
+    <gazebo reference="${prefix}finger_2">
+      <material>Gazebo/Grey</material>
+    </gazebo>
+    <joint name="${prefix}gripper_base_finger_2" type="prismatic">
+      <origin xyz="0.03 -0.037 0.001" rpy="0 0 0"/>
+      <parent link="${prefix}gripper_base"/>
+      <child link="${prefix}finger_2"/>
+      <axis xyz="0 1 0"/>
+      <limit effort="1.0" lower="0" upper="0.04" velocity="0.1"/>
+    </joint>
     <link name="${prefix}tool0" />
     <joint name="${prefix}flange-tool0" type="fixed">
@@ -270,4 +362,22 @@
       </actuator>
     </transmission>
+    <transmission name="${prefix}trans_gripper_finger_1">
+  <type>transmission_interface/SimpleTransmission</type>
+  <joint name="${prefix}gripper_base_finger_1">
+    <hardwareInterface>hardware_interface/PositionJointInterface</hardwareInterface>
+  </joint>
+  <actuator name="${prefix}motor_finger_1">
+    <mechanicalReduction>1</mechanicalReduction>
+  </actuator>
+</transmission>
+<transmission name="${prefix}trans_gripper_finger_2">
+  <type>transmission_interface/SimpleTransmission</type>
+  <joint name="${prefix}gripper_base_finger_2">
+    <hardwareInterface>hardware_interface/PositionJointInterface</hardwareInterface>
+  </joint>
+  <actuator name="${prefix}motor_finger_2">
+    <mechanicalReduction>1</mechanicalReduction>
+  </actuator>
+</transmission>
     <!-- Anchor to Gazebo world -->
     <gazebo reference="${prefix}base_link">
