Commit message: dinamica en rviz

File: fanuc_robot/fanuc_lrmate200id_support/urdf/lrmate200id.xacro (robot description, xacro)
@@ -1,5 +1,14 @@
 <?xml version="1.0"?>
 <robot name="fanuc_lrmate200id" xmlns:xacro="http://wiki.ros.org/xacro">
-  <xacro:include filename="$(find fanuc_lrmate200id_support)/urdf/lrmate200id_macro.xacro"/>
-  <xacro:fanuc_lrmate200id prefix=""/>
+  <!-- Declaramos el argumento -->
+  <xacro:arg name="modo_dinamico" default="true"/>
+  <!-- Usa el argumento directamente con $(arg …) -->
+  <xacro:if value="$(arg modo_dinamico)">
+    <xacro:include filename="$(find fanuc_lrmate200id_support)/urdf/lrmate200id_macro_din.xacro"/>
+    <xacro:fanuc_lrmate200id prefix=""/>
+  </xacro:if>
+  <xacro:unless value="$(arg modo_dinamico)">
+    <xacro:include filename="$(find fanuc_lrmate200id_support)/urdf/lrmate200id_macro.xacro"/>
+    <xacro:fanuc_lrmate200id prefix=""/>
+  </xacro:unless>
 </robot>

File: fanuc_robot/fanuc_lrmate200id_support/urdf/lrmate200id_macro_din.xacro (robot description, xacro)
@@ -145,5 +145,4 @@
       </collision>
     </link>
-    <!-- joints: main serial chain -->
     <joint name="${prefix}joint_1" type="revolute">
       <origin xyz="0 0 0.330" rpy="0 0 0" />
@@ -152,4 +151,5 @@
       <axis xyz="0 0 1" />
       <limit effort="30" lower="${radians(-170)}" upper="${radians(170)}" velocity="${radians(450)}" />
+      <dynamics damping="0.1" friction="0.0"/>
     </joint>
     <joint name="${prefix}joint_2" type="revolute">
@@ -159,4 +159,5 @@
       <axis xyz="0 1 0" />
       <limit effort="30" lower="${radians(-100)}" upper="${radians(145)}" velocity="${radians(380)}" />
+      <dynamics damping="0.1" friction="0.0"/>
     </joint>
     <joint name="${prefix}joint_3" type="revolute">
@@ -166,4 +167,5 @@
       <axis xyz="0 -1 0" />
       <limit effort="30" lower="${radians(-70)}" upper="${radians(205)}" velocity="${radians(520)}" />
+      <dynamics damping="0.1" friction="0.0"/>
     </joint>
     <joint name="${prefix}joint_4" type="revolute">
@@ -173,4 +175,5 @@
       <axis xyz="-1 0 0"/>
       <limit effort="20" lower="${radians(-190)}" upper="${radians(190)}" velocity="${radians(550)}" />
+      <dynamics damping="0.1" friction="0.0"/>
     </joint>
     <joint name="${prefix}joint_5" type="revolute">
@@ -180,4 +183,5 @@
       <axis xyz="0 -1 0"/>
       <limit effort="20" lower="${radians(-125)}" upper="${radians(125)}" velocity="${radians(545)}" />
+      <dynamics damping="0.1" friction="0.0"/>
     </joint>
     <joint name="${prefix}joint_6" type="revolute">
@@ -187,4 +191,5 @@
       <axis xyz="-1 0 0"/>
       <limit effort="10" lower="${radians(-360)}" upper="${radians(360)}" velocity="${radians(1000)}" />
+      <dynamics damping="0.1" friction="0.0"/>
     </joint>
     <!-- ROS-Industrial 'base' frame -->
@@ -258,6 +263,7 @@
       <parent link="${prefix}gripper_base"/>
       <child link="${prefix}finger_1"/>
-      <axis xyz="0 -1 0"/>   <!-- Cambia a -1 -->
+      <axis xyz="0 -1 0"/>
       <limit effort="1.0" lower="0" upper="0.04" velocity="0.1"/>
+      <dynamics damping="0.01" friction="0.0"/>
     </joint>
     <!-- Dedo derecho (finger_2) -->
@@ -293,4 +299,5 @@
       <axis xyz="0 1 0"/>
       <limit effort="1.0" lower="0" upper="0.04" velocity="0.1"/>
+      <dynamics damping="0.01" friction="0.0"/>
     </joint>
     <link name="${prefix}tool0" />
@@ -306,9 +313,9 @@
       </plugin>
     </gazebo>
-    <!-- Transmissions -->
+    <!-- Transmissions (brazo con esfuerzo) -->
     <transmission name="${prefix}trans_joint_1">
       <type>transmission_interface/SimpleTransmission</type>
       <joint name="${prefix}joint_1">
-        <hardwareInterface>hardware_interface/PositionJointInterface</hardwareInterface>
+        <hardwareInterface>hardware_interface/EffortJointInterface</hardwareInterface>
       </joint>
       <actuator name="${prefix}motor_joint_1">
@@ -316,9 +323,8 @@
       </actuator>
     </transmission>
-    <!-- Repite para los demás joints -->
     <transmission name="${prefix}trans_joint_2">
       <type>transmission_interface/SimpleTransmission</type>
       <joint name="${prefix}joint_2">
-        <hardwareInterface>hardware_interface/PositionJointInterface</hardwareInterface>
+        <hardwareInterface>hardware_interface/EffortJointInterface</hardwareInterface>
       </joint>
       <actuator name="${prefix}motor_joint_2">
@@ -329,5 +335,5 @@
       <type>transmission_interface/SimpleTransmission</type>
       <joint name="${prefix}joint_3">
-        <hardwareInterface>hardware_interface/PositionJointInterface</hardwareInterface>
+        <hardwareInterface>hardware_interface/EffortJointInterface</hardwareInterface>
       </joint>
       <actuator name="${prefix}motor_joint_3">
@@ -338,5 +344,5 @@
       <type>transmission_interface/SimpleTransmission</type>
       <joint name="${prefix}joint_4">
-        <hardwareInterface>hardware_interface/PositionJointInterface</hardwareInterface>
+        <hardwareInterface>hardware_interface/EffortJointInterface</hardwareInterface>
       </joint>
       <actuator name="${prefix}motor_joint_4">
@@ -347,5 +353,5 @@
       <type>transmission_interface/SimpleTransmission</type>
       <joint name="${prefix}joint_5">
-        <hardwareInterface>hardware_interface/PositionJointInterface</hardwareInterface>
+        <hardwareInterface>hardware_interface/EffortJointInterface</hardwareInterface>
       </joint>
       <actuator name="${prefix}motor_joint_5">
@@ -356,5 +362,5 @@
       <type>transmission_interface/SimpleTransmission</type>
       <joint name="${prefix}joint_6">
-        <hardwareInterface>hardware_interface/PositionJointInterface</hardwareInterface>
+        <hardwareInterface>hardware_interface/EffortJointInterface</hardwareInterface>
       </joint>
       <actuator name="${prefix}motor_joint_6">
@@ -362,22 +368,23 @@
       </actuator>
     </transmission>
+    <!-- Transmisiones del gripper (modo esfuerzo) -->
     <transmission name="${prefix}trans_gripper_finger_1">
-  <type>transmission_interface/SimpleTransmission</type>
-  <joint name="${prefix}gripper_base_finger_1">
-    <hardwareInterface>hardware_interface/PositionJointInterface</hardwareInterface>
-  </joint>
-  <actuator name="${prefix}motor_finger_1">
-    <mechanicalReduction>1</mechanicalReduction>
-  </actuator>
-</transmission>
-<transmission name="${prefix}trans_gripper_finger_2">
-  <type>transmission_interface/SimpleTransmission</type>
-  <joint name="${prefix}gripper_base_finger_2">
-    <hardwareInterface>hardware_interface/PositionJointInterface</hardwareInterface>
-  </joint>
-  <actuator name="${prefix}motor_finger_2">
-    <mechanicalReduction>1</mechanicalReduction>
-  </actuator>
-</transmission>
+      <type>transmission_interface/SimpleTransmission</type>
+      <joint name="${prefix}gripper_base_finger_1">
+        <hardwareInterface>hardware_interface/EffortJointInterface</hardwareInterface>
+      </joint>
+      <actuator name="${prefix}motor_finger_1">
+        <mechanicalReduction>1</mechanicalReduction>
+      </actuator>
+    </transmission>
+    <transmission name="${prefix}trans_gripper_finger_2">
+      <type>transmission_interface/SimpleTransmission</type>
+      <joint name="${prefix}gripper_base_finger_2">
+        <hardwareInterface>hardware_interface/EffortJointInterface</hardwareInterface>
+      </joint>
+      <actuator name="${prefix}motor_finger_2">
+        <mechanicalReduction>1</mechanicalReduction>
+      </actuator>
+    </transmission>
     <!-- Anchor to Gazebo world -->
     <gazebo reference="${prefix}base_link">
